Commit message: Mod: yaml file read in for gripper commands

File: urdf/inc/ur_common.xacro (robot description, xacro)
@@ -44,4 +44,6 @@
     <xacro:property name="config_physical_parameters" value="${xacro.load_yaml(physical_parameters_file)}"/>
     <xacro:property name="config_visual_parameters" value="${xacro.load_yaml(visual_parameters_file)}"/>
+    <xacro:property name="open_gripper_parameters" value="${xacro.load_yaml(open_gripper_script)}"/>
+    <xacro:property name="close_gripper_parameters" value="${xacro.load_yaml(close_gripper_script)}"/>
     <!-- Extract subsections from yaml dictionaries -->
     <xacro:property name="sec_limits" value="${config_joint_limit_parameters['joint_limits']}"/>
@@ -170,4 +172,7 @@
     <!--KINEMATICS HASH-->
     <xacro:property name="kinematics_hash" value="${sec_kinematics['hash']}" scope="parent"/>
+    <!--GRIPPER COMMANDS -->
+    <xacro:property name="open_gripper_command" value="${open_gripper_parameters['open_gripper']}" scope="parent"/>
+    <xacro:property name="close_gripper_command" value="${close_gripper_parameters['close_gripper']}" scope="parent"/>
   </xacro:macro>
 </robot>

File: urdf/ur_macro.xacro (robot description, xacro)
@@ -101,6 +101,6 @@
       sim_ignition="${sim_ignition}"
       script_filename="${script_filename}"
-      open_gripper_script="${open_gripper_script}"
-      close_gripper_script="${close_gripper_script}"
+      open_gripper_script="${open_gripper_command}"
+      close_gripper_script="${close_gripper_command}"
       output_recipe_filename="${output_recipe_filename}"
       input_recipe_filename="${input_recipe_filename}"

Commit message: Mod: parameter loading through yaml

File: urdf/inc/ur_common.xacro (robot description, xacro)
@@ -37,5 +37,5 @@
     <mesh filename="${mesh}"/>
   </xacro:macro>
-  <xacro:macro name="read_model_data" params="joint_limits_parameters_file kinematics_parameters_file physical_parameters_file visual_parameters_file force_abs_paths">
+  <xacro:macro name="read_model_data" params="joint_limits_parameters_file kinematics_parameters_file physical_parameters_file visual_parameters_file force_abs_paths open_gripper_script close_gripper_script">
     <xacro:property name="force_abs_paths" value="${force_abs_paths}" scope="parent"/>
     <!-- Read .yaml files from disk, load content into properties -->

File: urdf/ur_macro.xacro (robot description, xacro)
@@ -88,5 +88,7 @@
       physical_parameters_file="${physical_parameters_file}"
       visual_parameters_file="${visual_parameters_file}"
-      force_abs_paths="${sim_gazebo or sim_ignition}"/>
+      force_abs_paths="${sim_gazebo or sim_ignition}"
+      open_gripper_script="${open_gripper_script}"
+      close_gripper_script="${close_gripper_script}"/>
     <!-- ros2 control include -->
     <xacro:include filename="$(find ur_description)/urdf/ur.ros2_control.xacro" />
